File: pmod-dualrs422.sch (KiCad schematic (older format))
At the start: 14 parts, among them J1 Conn_02x06_Odd_Even, J2 Conn_01x10_Male, U1 MAX490E, U2 MAX490E

Commit message: Added Documentation/pmod-dualrs422.pdf
Other:
- note removed: "USE SIT3490\n"
Changed lines of the file:
@@
 Wire Wire Line
 	2850 3700 2600 3700
-Text Notes 5650 2150 0    118  ~ 0
-USE SIT3490\n
 Wire Wire Line
 	2100 3200 1550 3200
